Commit message: gazebo_simulation_env set up

File: turtlebot4_description/urdf/standard/turtlebot4.urdf.xacro (robot description, xacro)
@@ -9,7 +9,8 @@
   <xacro:include filename="$(find turtlebot4_description)/urdf/standard/tower_sensor_plate.urdf.xacro" />
   <xacro:include filename="$(find turtlebot4_description)/urdf/standard/weight_block.urdf.xacro" />
+  <!--
   <xacro:include filename="$(find turtlebot4_description)/urdf/body/body.urdf.xacro" />
-  <xacro:include filename="$(find turtlebot4_description)/urdf/arm/right_arm.urdf.xacro" />
-  <xacro:include filename="$(find turtlebot4_description)/urdf/arm/left_arm.urdf.xacro" />
+  <xacro:include filename="$(find turtlebot4_description)/urdf/arm/arm.urdf.xacro" />
+  -->
   <!-- Mechanical properties -->
   <xacro:property name="shell_z_offset"                value="${3*cm2m}" />
@@ -93,7 +94,13 @@
     <origin xyz="0 0 ${tower_sensor_plate_z_offset}"/>
   </xacro:tower_sensor_plate>
+  <!--
   <xacro:body name="body">
     <origin xyz="0 0 ${tower_standoff_z_offset+0.003}"/>
   </xacro:body>
+  <xacro:arm name="arm">
+    <origin xyz="0 0 0.17" rpy="0 0 ${3*pi/2}" />
+  </xacro:arm>
+   -->
+  <!--
   <xacro:right_arm name="right_arm">
     <origin xyz="0 0.06 0" rpy="${3*pi/2} ${3*pi/2} 0" />
@@ -102,4 +109,5 @@
     <origin xyz="0 -0.06 0" rpy="${pi/2} ${pi/2} 0" />
   </xacro:left_arm>
+   -->
   <!-- Turtlebot4 sensor definitions -->
   <xacro:rplidar name="rplidar" parent_link="shell_link" gazebo="$(arg gazebo)">
