Commit message: Added Moveit2 interfaces for AI

File: robotpi_demo_robot_description/urdf/arm/mycobot280.urdf.xacro (robot description, xacro)
@@ -443,4 +443,29 @@
 		<mimic joint="gripper_controller" multiplier="1.0" offset="0" />
 	</joint>
+	<link name="random1"/>
+	<link name="random2"/>
+	<link name="random3"/>
+	<link name="random4"/>
+	<link name="random5"/>
+    <joint name="gripper_base_to_gripper_left2_mimic" type="fixed">
+        <parent link="world"/>
+        <child link="random1"/>
+    </joint>
+	<joint name="gripper_left3_to_gripper_left1_mimic" type="fixed">
+        <parent link="world"/>
+        <child link="random2"/>
+    </joint>
+	<joint name="gripper_base_to_gripper_right3_mimic" type="fixed">
+        <parent link="world"/>
+        <child link="random3"/>
+    </joint>
+	<joint name="gripper_base_to_gripper_right2_mimic" type="fixed">
+        <parent link="world"/>
+        <child link="random4"/>
+    </joint>
+	<joint name="gripper_right3_to_gripper_right1_mimic" type="fixed">
+        <parent link="world"/>
+        <child link="random5"/>
+    </joint>
 	<gazebo reference="link1">
         <material>Gazebo/White</material>
@@ -467,3 +492,21 @@
         <material>Gazebo/White</material>
     </gazebo>
+	<gazebo reference="gripper_left1">
+        <material>Gazebo/White</material>
+    </gazebo>
+	<gazebo reference="gripper_left2">
+        <material>Gazebo/White</material>
+    </gazebo>
+	<gazebo reference="gripper_left3">
+        <material>Gazebo/White</material>
+    </gazebo>
+	<gazebo reference="gripper_right1">
+        <material>Gazebo/White</material>
+    </gazebo>
+	<gazebo reference="gripper_right2">
+        <material>Gazebo/White</material>
+    </gazebo>
+	<gazebo reference="gripper_right3">
+        <material>Gazebo/White</material>
+    </gazebo>
 </robot>

File: robotpi_demo_robot_description/urdf/arm/panda.urdf.xacro (robot description, xacro)
@@ -244,5 +244,5 @@
         </inertial>
   </link>
-    <joint name="panda_joint_world" type="fixed">
+    <joint name="virtual_joint" type="fixed">
         <parent link="world"/>
         <child link="panda_link0"/>
@@ -322,5 +322,5 @@
         <axis xyz="0 -1 0"/>
         <limit effort="20." lower="-0.001" upper="0.04" velocity="0.3"/>
-        <mimic joint="panda_finger_joint1" />
+        <mimic joint="panda_finger_joint1" multiplier="1.0"/>
     </joint>
     <joint name="end_effector_frame_fixed_joint" type="fixed">
@@ -329,4 +329,35 @@
         <child link="end_effector_frame"/>
     </joint>
+    <link name="random"/>
+    <joint name="panda_finger_joint2_mimic" type="fixed">
+        <parent link="world"/>
+        <child link="random"/>
+    </joint>
+    <!--
+    <link name="camera">
+        <visual>
+            <geometry>
+                <box size="0.05 0.05 0.05"/>
+            </geometry>
+        </visual>
+        <collision>
+            <geometry>
+                <box size="0.05 0.05 0.05"/>
+            </geometry>
+        </collision>
+        <inertial>
+            <mass value="0.1"/>
+            <origin xyz="0 0 0"/>
+            <inertia ixx="0.000001" ixy="0.0" ixz="0.0"
+                     iyy="0.000001" iyz="0.0"
+                     izz="0.000002"/>
+        </inertial>
+    </link>
+    <joint name="camera_to_panda_link0" type="fixed">
+        <parent link="world"/>
+        <child link="camera"/>
+        <origin xyz="0.5 -0.5 0" rpy="0.0 0.0 0.0"/>
+    </joint>
+     -->
     <gazebo reference="panda_link0">
       <material>Gazebo/White</material>
@@ -365,3 +396,8 @@
       <material>Gazebo/Black</material>
     </gazebo>
+    <!--
+    <gazebo reference="camera">
+        <material>Gazebo/Red</material>
+    </gazebo>
+     -->
 </robot>
