Commit message: Failed to accomplish pick and place

File: robotpi_demo_robot_description/urdf/arm/panda.urdf.xacro (robot description, xacro)
@@ -3,4 +3,13 @@
     <xacro:include filename="$(find robotpi_demo_robot_description)/urdf/ros2_control/panda/panda_gazebo_ros2_control.xacro"/>
 	<xacro:include filename="$(find robotpi_demo_robot_description)/urdf/ros2_control/panda/panda_ros2_control.xacro"/>
+    <xacro:macro name="default_transmission" params="joint_name">
+        <transmission name="transmission_${joint_name}">
+            <plugin>transmission_interface/SimpleTransmission</plugin>
+            <actuator name="actuator_${joint_name}" role="actuator_${joint_name}"/>
+            <joint name="${joint_name}" role="${joint_name}">
+                <mechanical_reduction>1.0</mechanical_reduction>
+            </joint>
+        </transmission>
+    </xacro:macro>
   <link name="world"/>
   <link name="panda_link0">
@@ -213,4 +222,12 @@
                 <mesh filename="file://$(find robotpi_demo_robot_description)/meshes/panda/collision/finger.stl"/>
             </geometry>
+            <surface>
+                <friction>
+                    <ode>
+                        <mu>5.0</mu> <!-- 静摩擦系数 -->
+                        <mu2>5.0</mu2> <!-- 动摩擦系数 -->
+                    </ode>
+                </friction>
+            </surface>
         </collision>
   </link>
@@ -234,6 +251,15 @@
                 <mesh filename="file://$(find robotpi_demo_robot_description)/meshes/panda/collision/finger.stl"/>
             </geometry>
-        </collision>
-  </link>
+            <surface>
+                <friction>
+                    <ode>
+                        <mu>5.0</mu> <!-- 静摩擦系数 -->
+                        <mu2>5.0</mu2> <!-- 动摩擦系数 -->
+                    </ode>
+                </friction>
+            </surface>
+        </collision>
+  </link>
+  <!--
   <link name="end_effector_frame">
         <inertial>
@@ -244,5 +270,6 @@
         </inertial>
   </link>
-    <joint name="virtual_joint" type="fixed">
+ -->
+    <joint name="world_joint" type="fixed">
         <parent link="world"/>
         <child link="panda_link0"/>
@@ -314,5 +341,5 @@
         <origin rpy="0 0 0" xyz="0 0 0.0584"/>
         <axis xyz="0 1 0"/>
-        <limit effort="20." lower="-0.001" upper="0.04" velocity="0.3"/>
+        <limit effort="5000." lower="-0.001" upper="0.04" velocity="0.3"/>
     </joint>
     <joint name="panda_finger_joint2" type="prismatic">
@@ -321,7 +348,8 @@
         <origin rpy="0 0 0" xyz="0 0 0.0584"/>
         <axis xyz="0 -1 0"/>
-        <limit effort="20." lower="-0.001" upper="0.04" velocity="0.3"/>
-        <mimic joint="panda_finger_joint1" multiplier="1.0"/>
-    </joint>
+        <limit effort="5000." lower="-0.001" upper="0.04" velocity="0.3"/>
+        <!-- <mimic joint="panda_finger_joint1" multiplier="1.0"/> -->
+    </joint>
+    <!--
     <joint name="end_effector_frame_fixed_joint" type="fixed">
         <origin rpy="3.14159 -1.57079 -0.785398163397" xyz="0 0 0.21"/>
@@ -329,35 +357,10 @@
         <child link="end_effector_frame"/>
     </joint>
-    <link name="random"/>
+     -->
+    <!-- <link name="random"/>
     <joint name="panda_finger_joint2_mimic" type="fixed">
         <parent link="world"/>
         <child link="random"/>
-    </joint>
-    <!--
-    <link name="camera">
-        <visual>
-            <geometry>
-                <box size="0.05 0.05 0.05"/>
-            </geometry>
-        </visual>
-        <collision>
-            <geometry>
-                <box size="0.05 0.05 0.05"/>
-            </geometry>
-        </collision>
-        <inertial>
-            <mass value="0.1"/>
-            <origin xyz="0 0 0"/>
-            <inertia ixx="0.000001" ixy="0.0" ixz="0.0"
-                     iyy="0.000001" iyz="0.0"
-                     izz="0.000002"/>
-        </inertial>
-    </link>
-    <joint name="camera_to_panda_link0" type="fixed">
-        <parent link="world"/>
-        <child link="camera"/>
-        <origin xyz="0.5 -0.5 0" rpy="0.0 0.0 0.0"/>
-    </joint>
-     -->
+    </joint> -->
     <gazebo reference="panda_link0">
       <material>Gazebo/White</material>
@@ -396,8 +399,12 @@
       <material>Gazebo/Black</material>
     </gazebo>
-    <!--
-    <gazebo reference="camera">
-        <material>Gazebo/Red</material>
-    </gazebo>
-     -->
+    <xacro:default_transmission joint_name="panda_joint1"/>
+    <xacro:default_transmission joint_name="panda_joint2"/>
+    <xacro:default_transmission joint_name="panda_joint3"/>
+    <xacro:default_transmission joint_name="panda_joint4"/>
+    <xacro:default_transmission joint_name="panda_joint5"/>
+    <xacro:default_transmission joint_name="panda_joint6"/>
+    <xacro:default_transmission joint_name="panda_joint7"/>
+    <xacro:default_transmission joint_name="panda_finger_joint1"/>
+    <xacro:default_transmission joint_name="panda_finger_joint2"/>
 </robot>

File: robotpi_demo_robot_description/urdf/ros2_control/panda/panda_ros2_control.xacro (robot description, xacro)
@@ -6,7 +6,8 @@
         </hardware>
         <joint name="panda_joint1">
-            <command_interface name="position">
-                <param name="min">-2.879793</param>
-                <param name="max">2.879793</param>
+            <command_interface name="position"/>
+            <command_interface name="effort">
+              <param name="min">-500</param>
+              <param name="max">500</param>
             </command_interface>
             <state_interface name="position"/>
@@ -15,4 +16,8 @@
         <joint name="panda_joint2">
             <command_interface name="position"/>
+            <command_interface name="effort">
+              <param name="min">-500</param>
+              <param name="max">500</param>
+            </command_interface>
             <state_interface name="position">
               <param name="initial_value"> -0.785</param>
@@ -24,4 +29,8 @@
         <joint name="panda_joint3">
             <command_interface name="position"/>
+            <command_interface name="effort">
+              <param name="min">-500</param>
+              <param name="max">500</param>
+            </command_interface>
             <state_interface name="position">
               <param name="initial_value">0.0</param>
@@ -33,4 +42,8 @@
         <joint name="panda_joint4">
             <command_interface name="position"/>
+            <command_interface name="effort">
+              <param name="min">-500</param>
+              <param name="max">500</param>
+            </command_interface>
             <state_interface name="position">
               <param name="initial_value">-2.356</param>
@@ -42,4 +55,8 @@
         <joint name="panda_joint5">
             <command_interface name="position"/>
+            <command_interface name="effort">
+              <param name="min">-500</param>
+              <param name="max">500</param>
+            </command_interface>
             <state_interface name="position">
               <param name="initial_value">0.0</param>
@@ -51,4 +68,8 @@
         <joint name="panda_joint6">
             <command_interface name="position"/>
+            <command_interface name="effort">
+              <param name="min">-500</param>
+              <param name="max">500</param>
+            </command_interface>
             <state_interface name="position">
               <param name="initial_value">1.571</param>
@@ -60,4 +81,8 @@
         <joint name="panda_joint7">
             <command_interface name="position"/>
+            <command_interface name="effort">
+              <param name="min">-500</param>
+              <param name="max">500</param>
+            </command_interface>
             <state_interface name="position">
               <param name="initial_value">0.785</param>
@@ -68,22 +93,38 @@
         </joint>
         <joint name="panda_finger_joint1">
-            <command_interface name="position" />
+            <!-- <command_interface name="position"/> -->
+            <command_interface name="effort">
+              <param name="min">-500</param>
+              <param name="max">500</param>
+            </command_interface>
             <state_interface name="position">
               <param name="initial_value">0.0</param>
             </state_interface>
-            <state_interface name="velocity">
-                <param name="initial_value">0.0</param>
-            </state_interface>
-        </joint>
-        <joint name="panda_finger_joint2">
-            <param name="mimic">panda_finger_joint1</param>
-            <param name="multiplier">1</param>
-            <command_interface name="position" />
-            <state_interface name="position">
+            <state_interface name="effort">
               <param name="initial_value">0.0</param>
             </state_interface>
             <state_interface name="velocity">
-                <param name="initial_value">0.0</param>
+              <param name="initial_value">0.0</param>
             </state_interface>
+            <dynamics damping="0.2" friction="0.1"/>
+        </joint>
+        <joint name="panda_finger_joint2">
+          <!-- <param name="mimic">panda_finger_joint1</param>
+          <param name="multiplier">1</param> -->
+          <!-- <command_interface name="position"/> -->
+          <command_interface name="effort">
+            <param name="min">-500</param>
+            <param name="max">500</param>
+          </command_interface>
+          <state_interface name="position">
+            <param name="initial_value">0.0</param>
+          </state_interface>
+          <state_interface name="effort">
+            <param name="initial_value">0.0</param>
+          </state_interface>
+          <state_interface name="velocity">
+            <param name="initial_value">0.0</param>
+          </state_interface>
+          <dynamics damping="0.2" friction="0.1"/>
         </joint>
     </ros2_control>

Commit message: Modified ros2 control yaml file

File: robotpi_demo_robot_description/urdf/arm/panda.urdf.xacro (robot description, xacro)
@@ -349,5 +349,5 @@
         <axis xyz="0 -1 0"/>
         <limit effort="5000." lower="-0.001" upper="0.04" velocity="0.3"/>
-        <!-- <mimic joint="panda_finger_joint1" multiplier="1.0"/> -->
+        <mimic joint="panda_finger_joint1" multiplier="1.0"/>
     </joint>
     <!--
@@ -358,43 +358,55 @@
     </joint>
      -->
-    <!-- <link name="random"/>
+    <link name="random"/>
     <joint name="panda_finger_joint2_mimic" type="fixed">
         <parent link="world"/>
         <child link="random"/>
-    </joint> -->
+    </joint>
     <gazebo reference="panda_link0">
+      <selfCollide>false</selfCollide>
       <material>Gazebo/White</material>
     </gazebo>
     <gazebo reference="panda_link1">
+      <selfCollide>false</selfCollide>
       <material>Gazebo/White</material>
     </gazebo>
     <gazebo reference="panda_link2">
+      <selfCollide>false</selfCollide>
       <material>Gazebo/White</material>
     </gazebo>
     <gazebo reference="panda_link3">
+      <selfCollide>false</selfCollide>
       <material>Gazebo/White</material>
     </gazebo>
     <gazebo reference="panda_link4">
+      <selfCollide>false</selfCollide>
       <material>Gazebo/White</material>
     </gazebo>
     <gazebo reference="panda_link5">
+      <selfCollide>false</selfCollide>
       <material>Gazebo/White</material>
     </gazebo>
     <gazebo reference="panda_link6">
+      <selfCollide>false</selfCollide>
       <material>Gazebo/White</material>
     </gazebo>
     <gazebo reference="panda_link7">
+      <selfCollide>false</selfCollide>
       <material>Gazebo/White</material>
     </gazebo>
     <gazebo reference="panda_link8">
+      <selfCollide>false</selfCollide>
       <material>Gazebo/White</material>
     </gazebo>
     <gazebo reference="panda_hand">
+      <selfCollide>false</selfCollide>
       <material>Gazebo/White</material>
     </gazebo>
     <gazebo reference="panda_leftfinger">
+      <selfCollide>false</selfCollide>
       <material>Gazebo/Black</material>
     </gazebo>
     <gazebo reference="panda_rightfinger">
+      <selfCollide>false</selfCollide>
       <material>Gazebo/Black</material>
     </gazebo>
@@ -407,4 +419,3 @@
     <xacro:default_transmission joint_name="panda_joint7"/>
     <xacro:default_transmission joint_name="panda_finger_joint1"/>
-    <xacro:default_transmission joint_name="panda_finger_joint2"/>
 </robot>

File: robotpi_demo_robot_description/urdf/ros2_control/panda/panda_ros2_control.xacro (robot description, xacro)
@@ -6,5 +6,5 @@
         </hardware>
         <joint name="panda_joint1">
-            <command_interface name="position"/>
+            <!-- <command_interface name="position"/> -->
             <command_interface name="effort">
               <param name="min">-500</param>
@@ -15,5 +15,5 @@
         </joint>
         <joint name="panda_joint2">
-            <command_interface name="position"/>
+            <!-- <command_interface name="position"/> -->
             <command_interface name="effort">
               <param name="min">-500</param>
@@ -28,5 +28,5 @@
         </joint>
         <joint name="panda_joint3">
-            <command_interface name="position"/>
+            <!-- <command_interface name="position"/> -->
             <command_interface name="effort">
               <param name="min">-500</param>
@@ -41,5 +41,5 @@
         </joint>
         <joint name="panda_joint4">
-            <command_interface name="position"/>
+            <!-- <command_interface name="position"/> -->
             <command_interface name="effort">
               <param name="min">-500</param>
@@ -54,5 +54,5 @@
         </joint>
         <joint name="panda_joint5">
-            <command_interface name="position"/>
+            <!-- <command_interface name="position"/> -->
             <command_interface name="effort">
               <param name="min">-500</param>
@@ -67,5 +67,5 @@
         </joint>
         <joint name="panda_joint6">
-            <command_interface name="position"/>
+            <!-- <command_interface name="position"/> -->
             <command_interface name="effort">
               <param name="min">-500</param>
@@ -80,5 +80,5 @@
         </joint>
         <joint name="panda_joint7">
-            <command_interface name="position"/>
+            <!-- <command_interface name="position"/> -->
             <command_interface name="effort">
               <param name="min">-500</param>
@@ -101,10 +101,8 @@
               <param name="initial_value">0.0</param>
             </state_interface>
-            <state_interface name="effort">
-              <param name="initial_value">0.0</param>
-            </state_interface>
             <state_interface name="velocity">
               <param name="initial_value">0.0</param>
             </state_interface>
+            <state_interface name="effort"/>
             <dynamics damping="0.2" friction="0.1"/>
         </joint>
@@ -120,10 +118,8 @@
             <param name="initial_value">0.0</param>
           </state_interface>
-          <state_interface name="effort">
-            <param name="initial_value">0.0</param>
-          </state_interface>
           <state_interface name="velocity">
             <param name="initial_value">0.0</param>
           </state_interface>
+          <state_interface name="effort"/>
           <dynamics damping="0.2" friction="0.1"/>
         </joint>

Commit message: can do pick and place using mtc in rviz

File: robotpi_demo_robot_description/urdf/arm/panda.urdf.xacro (robot description, xacro)
@@ -236,5 +236,5 @@
         </collision>
   </link>
-  <link name="end_effector_frame">
+  <!-- <link name="end_effector_frame">
         <inertial>
             <mass value="0.01"/>
@@ -243,5 +243,5 @@
                 iyy="0.0001" iyz="0.0" izz="0.0001"/>
         </inertial>
-  </link>
+  </link> -->
     <joint name="virtual_joint" type="fixed">
         <parent link="world"/>
@@ -324,5 +324,5 @@
         <mimic joint="panda_finger_joint1" multiplier="1.0"/>
     </joint>
-    <joint name="end_effector_frame_fixed_joint" type="fixed">
+    <!-- <joint name="end_effector_frame_fixed_joint" type="fixed">
         <origin rpy="3.14159 -1.57079 -0.785398163397" xyz="0 0 0.21"/>
         <parent link="panda_link7"/>
@@ -333,5 +333,5 @@
         <parent link="world"/>
         <child link="random"/>
-    </joint>
+    </joint> -->
     <!--
     <link name="camera">

Commit message: update param for pick and play

File: robotpi_demo_robot_description/urdf/arm/panda.urdf.xacro (robot description, xacro)
@@ -236,5 +236,5 @@
         </collision>
   </link>
-  <!-- <link name="end_effector_frame">
+  <link name="end_effector_frame">
         <inertial>
             <mass value="0.01"/>
@@ -243,5 +243,5 @@
                 iyy="0.0001" iyz="0.0" izz="0.0001"/>
         </inertial>
-  </link> -->
+  </link>
     <joint name="virtual_joint" type="fixed">
         <parent link="world"/>
@@ -324,5 +324,5 @@
         <mimic joint="panda_finger_joint1" multiplier="1.0"/>
     </joint>
-    <!-- <joint name="end_effector_frame_fixed_joint" type="fixed">
+    <joint name="end_effector_frame_fixed_joint" type="fixed">
         <origin rpy="3.14159 -1.57079 -0.785398163397" xyz="0 0 0.21"/>
         <parent link="panda_link7"/>
@@ -333,5 +333,5 @@
         <parent link="world"/>
         <child link="random"/>
-    </joint> -->
+    </joint>
     <!--
     <link name="camera">

Commit message: Moveit can't specify desired effort for effort controller

File: robotpi_demo_robot_description/urdf/arm/panda.urdf.xacro (robot description, xacro)
@@ -3,4 +3,7 @@
     <xacro:include filename="$(find robotpi_demo_robot_description)/urdf/ros2_control/panda/panda_gazebo_ros2_control.xacro"/>
 	<xacro:include filename="$(find robotpi_demo_robot_description)/urdf/ros2_control/panda/panda_ros2_control.xacro"/>
+    <xacro:property name="joint_effort" value="56.0"/>
+    <xacro:property name="joint_damping" value="0.0"/>
+    <xacro:property name="joint_friction" value="0.0"/>
   <link name="world"/>
   <link name="panda_link0">
@@ -308,4 +311,5 @@
         <child link="panda_hand"/>
         <origin rpy="0 0 -0.785398163397" xyz="0 0 0"/>
+        <dynamics damping="${joint_damping}" friction="${joint_friction}"/>
     </joint>
     <joint name="panda_finger_joint1" type="prismatic">
@@ -315,4 +319,5 @@
         <axis xyz="0 1 0"/>
         <limit effort="20." lower="-0.001" upper="0.04" velocity="0.3"/>
+        <dynamics damping="${joint_damping}" friction="${joint_friction}"/>
     </joint>
     <joint name="panda_finger_joint2" type="prismatic">
@@ -322,4 +327,5 @@
         <axis xyz="0 -1 0"/>
         <limit effort="20." lower="-0.001" upper="0.04" velocity="0.3"/>
+        <dynamics damping="${joint_damping}" friction="${joint_friction}"/>
         <mimic joint="panda_finger_joint1" multiplier="1.0"/>
     </joint>
@@ -334,4 +340,22 @@
         <child link="random"/>
     </joint>
+    <!-- <transmission name="panda_finger_trans1">
+        <type>transmission_interface/SimpleTransmission</type>
+        <joint name="panda_finger_joint1">
+            <hardwareInterface>EffortJointInterface</hardwareInterface>
+        </joint>
+        <actuator name="panda_finger_motor1">
+            <mechanicalReduction>1</mechanicalReduction>
+        </actuator>
+    </transmission>
+        <transmission name="panda_finger_trans2">
+        <type>transmission_interface/SimpleTransmission</type>
+        <joint name="panda_finger_joint2">
+            <hardwareInterface>EffortJointInterface</hardwareInterface>
+        </joint>
+        <actuator name="panda_finger_motor2">
+            <mechanicalReduction>1</mechanicalReduction>
+        </actuator>
+    </transmission> -->
     <!--
     <link name="camera">

File: robotpi_demo_robot_description/urdf/ros2_control/panda/panda_ros2_control.xacro (robot description, xacro)
@@ -79,5 +79,4 @@
             <param name="mimic">panda_finger_joint1</param>
             <param name="multiplier">1</param>
-            <command_interface name="position" />
             <state_interface name="position">
               <param name="initial_value">0.0</param>
